File: ChargerAndPowerSupply/ChargerAndPowerSupply.kicad_pcb (KiCad board)
At the start: 2 copper layers, 111.8 x 71.1 mm, 24 parts, among them IC1 LM2576T-005G, J1 16VAC, J2 +12 G PF +5 G, J3 + Battery -, U1 LM317K, U2 VO615A-6

Commit message: Minor update -- footprints and 3D shapes.
Parts:
- IC1: footprint LM2576T-005G:MC34166TG -> TO_SOT_Packages_THT:TO-220-5_Pentawatt_Multiwatt-5_Vertical_StaggeredType1
- L1: footprint PE-53113NL:PE53113NL -> Inductors_THT:L_Toroid_Vertical_L24.6mm_W15.5mm_P11.44mm_Pulse_KM-4
- moved MK2 12.5 mm to (119.6, 160.0)
- moved MK3 12.5 mm to (119.6, 99.1)
- moved IC1 0.29 mm to (38.0, 146.5)
- moved L1 0.18 mm to (63.5, 135.9)
Routing:
- net Net-(D2-Pad1): track 31.6 -> 35.3 mm
