File: ChargerAndPowerSupply/ChargerAndPowerSupply.kicad_pcb (KiCad board)
At the start: 2 copper layers, 111.8 x 71.1 mm, 24 parts, among them IC1 LM2576T-005G, J1 16VAC, J2 +12 G PF +5 G, J3 + Battery -, U1 LM317K, U2 VO615A-6

Commit message: Upgrade KiCAD files.
Other:
- net class Default removed
