File: ChargerAndPowerSupply/ChargerAndPowerSupply.sch (KiCad schematic (older format))
At the start: 24 parts, among them IC1 LM2576T-005G, J1 16VAC, J2 +12 G PF +5 G, J3 + Battery -, U1 LM317K, U2 VO615A-6

Commit message: Minor update -- footprints and 3D shapes.
Parts:
- IC1: footprint LM2576T-005G:MC34166TG -> TO_SOT_Packages_THT:TO-220-5_Pentawatt_Multiwatt-5_Vertical_StaggeredType1
- L1: footprint PE-53113NL:PE53113NL -> Inductors_THT:L_Toroid_Vertical_L24.6mm_W15.5mm_P11.44mm_Pulse_KM-4
Changed lines of the file:
@@
 F 0 "IC1" H 4800 6350 50  0000 L CNN
 F 1 "LM2576T-005G" H 4800 6250 50  0000 L CNN
-F 2 "LM2576T-005G:MC34166TG" H 4800 6150 50  0001 L CNN
+F 2 "TO_SOT_Packages_THT:TO-220-5_Pentawatt_Multiwatt-5_Vertical_StaggeredType1" H 4800 6150 50  0001 L CNN
 F 3 "https://componentsearchengine.com//LM2576T-005G.pdf" H 4800 6050 50  0001 L CNN
 F 4 "Buck Regulator, Switching, 3.0 A, 15 V 3.0 A, 5.0 V, 52 kHz" H 4800 5950 50  0001 L CNN "Description"
@@
 F 0 "L1" V 5100 6050 50  0000 L CNN
 F 1 "150uH" V 5150 5900 50  0000 L CNN
-F 2 "PE-53113NL:PE53113NL" H 5200 6050 50  0001 C CNN
+F 2 "Inductors_THT:L_Toroid_Vertical_L24.6mm_W15.5mm_P11.44mm_Pulse_KM-4" H 5200 6050 50  0001 C CNN
 F 3 "" H 5200 6050 50  0001 C CNN
 F 4 "673-PE-53113NL " V 5200 6050 60  0001 C CNN "Mouser Part Number"
