File: ChargerAndPowerSupply/ChargerAndPowerSupply.kicad_sch (KiCad schematic)
At the start: 24 parts, among them IC1 LM2576T-005G, J1 16VAC, J2 +12 G PF +5 G, J3 + Battery -, U1 LM317K, U2 VO615A-6

Commit message: Tweaks to the Charger PS.
Parts:
- D2, D4: Mouser Part Number (none) -> 511-1N5822-TR
- D3: Mouser Part Number (none) -> 621-SBR10U300CT
- IC1: Mouser Part Number (none) -> 863-LM2576T-005G; Mouser2 Part Number 863-LM2576T-005G -> (none)
- J1: Mouser Part Number (none) -> 651-1017491; Mouser Part Numer 651-1017491 -> (none)
- J2: Mouser Part Number (none) -> 538-26-60-7050
- J3: Mouser Part Number (none) -> 538-26-60-7020
- U1: Mouser Part Number LM317KCT -> 595-LM317KCS
- U2: Mouser Part Number (none) -> 78-VO615A-6
Changed lines of the file:
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@@
       (effects (font (size 1.27 1.27)) hide)
     )
-    (property "Mouser Part Number" "LM317KCT" (id 4) (at 116.84 68.58 0)
+    (property "Mouser Part Number" "595-LM317KCS " (id 4) (at 116.84 68.58 0)
       (effects (font (size 1.524 1.524)) hide)
     )
@@
       (effects (font (size 1.27 1.27)) hide)
     )
+    (property "Mouser Part Number" "621-SBR10U300CT" (id 4) (at 161.29 76.2 0)
+      (effects (font (size 1.27 1.27)) hide)
+    )
     (pin "1")
     (pin "2")
@@
       (effects (font (size 1.27 1.27)) hide)
     )
+    (property "Mouser Part Number" " 538-26-60-7020" (id 4) (at 185.42 83.82 0)
+      (effects (font (size 1.27 1.27)) hide)
+    )
     (pin "1")
     (pin "2")
@@
       (effects (font (size 1.27 1.27)) hide)
     )
+    (property "Mouser Part Number" "511-1N5822-TR" (id 4) (at 180.34 68.58 0)
+      (effects (font (size 1.27 1.27)) hide)
+    )
     (pin "1")
     (pin "2")
@@
       (effects (font (size 1.27 1.27)) hide)
     )
+    (property "Mouser Part Number" "78-VO615A-6" (id 4) (at 163.83 62.23 0)
+      (effects (font (size 1.27 1.27)) hide)
+    )
     (pin "1")
     (pin "2")
@@
       (effects (font (size 1.27 1.27)) hide)
     )
-    (property "Mouser Part Numer" "651-1017491" (id 4) (at 38.1 67.31 0)
+    (property "Mouser Part Number" "651-1017491" (id 4) (at 38.1 67.31 0)
       (effects (font (size 1.524 1.524)) hide)
     )
@@
       (effects (font (size 1.27 1.27)) (justify left) hide)
     )
-    (property "Mouser2 Part Number" "863-LM2576T-005G" (id 6) (at 121.92 161.29 0)
+    (property "Mouser Part Number" "863-LM2576T-005G" (id 6) (at 121.92 161.29 0)
       (effects (font (size 1.27 1.27)) (justify left) hide)
     )
@@
       (effects (font (size 1.27 1.27)) hide)
     )
+    (property "Mouser Part Number" "511-1N5822-TR" (id 4) (at 128.27 162.56 0)
+      (effects (font (size 1.27 1.27)) hide)
+    )
     (pin "1")
     (pin "2")
@@
       (effects (font (size 1.27 1.27)) hide)
     )
+    (property "Mouser Part Number" "538-26-60-7050" (id 4) (at 162.56 143.51 0)
+      (effects (font (size 1.27 1.27)) hide)
+    )
